File: product_display_stepper_speaker/Circuit/V1/Circuit_final_design.kicad_sch (KiCad schematic)
At the start: 21 parts, among them J1 Barrel_Jack_MountingPin, U1 L7805, U2 LD33v, U3 ESP-12E

Commit message: started V2 of this project, gonna use Pico w instead of esp-12e
Other:
- note added: "the GPIO15 isn't grounded which it should,"
- note added: "the circuit was unstable and the MCU only booted proper when a semi-working DRV8825 driver was connected to first or second slot"
Changed lines of the file:
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@@
+		)
+	)
+	(text "the GPIO15 isn't grounded which it should, "
+		(exclude_from_sim no)
+		(at 167.386 138.684 0)
+		(effects
+			(font
+				(size 1.27 1.27)
+			)
+		)
+	)
+	(text "the circuit was unstable and the MCU only booted proper when a semi-working DRV8825 driver was connected to first or second slot"
+		(exclude_from_sim no)
+		(at 170.18 150.368 0)
+		(effects
+			(font
+				(size 1.27 1.27)
+			)
 		)
 	)
