File: hospital_traversing_robot/Electronics/station_circuit/station_circuit.kicad_pcb (KiCad board)
At the start: 2 copper layers, 70.8 x 55.9 mm, 21 parts, among them J1 Barrel_Jack_MountingPin, SW1 switch, SW2 SW_Push, U1 Pico, U2 NRF24L01_Breakout, U3 LM338T

Commit message: started station programming
Parts:
- moved R1 8.27 mm to (156.8, 92.8), turned to 180 degrees
- moved R2 3.25 mm to (149.2, 89.7)
Connections:
- R1 pad 2: Net-(R1-Pad2) -> Net-(U3-ADJ)
- R2 pad 1: GND -> Net-(U3-ADJ)
- R2 pad 2: Net-(R1-Pad2) -> GND
- U3 pad 1: GND -> Net-(U3-ADJ)
Routing:
- net Net-(U3-ADJ): track 0.00 -> 7.43 mm
- net +3.3V: track 41.2 -> 34.6 mm
- net GND: track 139.8 -> 144.1 mm
- net Net-(R1-Pad2): track 3.20 -> 0.00 mm
