File: hospital_traversing_robot/Electronics/station_circuit/station_circuit.kicad_pcb (KiCad board)
At the start: 2 copper layers, 70.8 x 55.9 mm, 21 parts, among them J1 Barrel_Jack_MountingPin, SW1 switch, SW2 SW_Push, U1 Pico, U2 NRF24L01_Breakout, U3 LM338T

Commit message: further development in hospital rover project
Parts:
- removed SW1: switch, Connector_PinHeader_2.54mm:PinHeader_1x03_P2.54mm_Vertical
Connections:
- SW2 pad 2: GNDA -> Net-(SW2-Pad2)
- U1 pad 28: GNDA -> Net-(SW2-Pad2)
- U1 pad 36: +3.3VA -> unconnected-(U1-3V3-Pad36)
- U2 pad 1: GNDA -> GND
- U2 pad 2: +3.3VP -> +3.3V
Routing:
- net GND: track 144.1 -> 195.0 mm
- net +3.3VA: track 34.5 -> 0.00 mm
- net GNDA: track 24.4 -> 0.00 mm
- net +3.3VP: track 15.9 -> 0.00 mm
- net +3.3V: track 34.6 -> 50.3 mm
- net Net-(SW2-Pad2): track 0.00 -> 14.7 mm
- net unconnected-(U1-3V3-Pad36): track 0.00 -> 0.81 mm
