File: hospital_traversing_robot/Electronics/station_circuit/station_circuit.kicad_sch (KiCad schematic)
At the start: 21 parts, among them J1 Barrel_Jack_MountingPin, SW1 switch, SW2 SW_Push, U1 Pico, U2 NRF24L01_Breakout, U3 LM338T

Commit message: started station programming
Connections:
- net GND: now also R2.2; no longer R2.1, U3.1 (ADJ)
- net at R1.2: now also R2.1, U3.1 (ADJ); no longer R2.2
Other:
- moved on the sheet: R2
Changed lines of the file:
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@@
 	)
 	(junction
-		(at 80.01 68.58)
+		(at 80.01 67.31)
 		(diameter 0)
 		(color 0 0 0 0)
@@
 	(wire
 		(pts
-			(xy 93.98 64.77) (xy 93.98 68.58)
+			(xy 80.01 67.31) (xy 93.98 67.31)
 		)
 		(stroke
@@
 	(wire
 		(pts
-			(xy 93.98 55.88) (xy 93.98 57.15)
+			(xy 80.01 68.58) (xy 80.01 67.31)
 		)
 		(stroke
@@
 	(wire
 		(pts
-			(xy 156.21 105.41) (xy 165.1 105.41)
+			(xy 93.98 67.31) (xy 93.98 64.77)
 		)
 		(stroke
@@
 	(wire
 		(pts
-			(xy 161.29 95.25) (xy 165.1 95.25)
+			(xy 93.98 55.88) (xy 93.98 57.15)
 		)
 		(stroke
@@
 	(wire
 		(pts
-			(xy 92.71 55.88) (xy 93.98 55.88)
+			(xy 156.21 105.41) (xy 165.1 105.41)
 		)
 		(stroke
@@
 	(wire
 		(pts
-			(xy 93.98 55.88) (xy 95.25 55.88)
+			(xy 161.29 95.25) (xy 165.1 95.25)
 		)
 		(stroke
@@
 	(wire
 		(pts
-			(xy 80.01 68.58) (xy 86.36 68.58)
+			(xy 92.71 55.88) (xy 93.98 55.88)
 		)
 		(stroke
@@
 	(wire
 		(pts
-			(xy 80.01 67.31) (xy 80.01 68.58)
-		)
-		(stroke
-			(width 0)
-			(type default)
-		)
-	)
-	(wire
-		(pts
-			(xy 80.01 68.58) (xy 80.01 71.12)
+			(xy 93.98 55.88) (xy 95.25 55.88)
 		)
 		(stroke
@@
 	(symbol
 		(lib_id "power:GND")
-		(at 80.01 71.12 0)
+		(at 80.01 76.2 0)
 		(unit 1)
 		(exclude_from_sim no)
@@
 		(fields_autoplaced yes)
 		(property "Reference" "#PWR02"
-			(at 80.01 77.47 0)
+			(at 80.01 82.55 0)
 			(effects
 				(font
@@
 		)
 		(property "Value" "GND"
+			(at 80.01 81.28 0)
+			(effects
+				(font
+					(size 1.27 1.27)
+				)
+			)
+		)
+		(property "Footprint" ""
 			(at 80.01 76.2 0)
 			(effects
@@
 					(size 1.27 1.27)
 				)
-			)
-		)
-		(property "Footprint" ""
-			(at 80.01 71.12 0)
-			(effects
-				(font
-					(size 1.27 1.27)
-				)
 				(hide yes)
 			)
 		)
 		(property "Datasheet" ""
-			(at 80.01 71.12 0)
+			(at 80.01 76.2 0)
 			(effects
 				(font
@@
 		)
 		(property "Description" "Power symbol creates a global label with name \"GND\" , ground"
-			(at 80.01 71.12 0)
+			(at 80.01 76.2 0)
 			(effects
 				(font
@@
 	(symbol
 		(lib_id "Device:R")
-		(at 90.17 68.58 90)
+		(at 80.01 72.39 0)
 		(unit 1)
 		(exclude_from_sim no)
@@
 		(dnp no)
 		(property "Reference" "R2"
-			(at 90.17 63.754 90)
+			(at 84.836 72.39 90)
 			(effects
 				(font
@@
 		)
 		(property "Value" "330"
-			(at 90.17 66.294 90)
+			(at 82.296 72.39 90)
 			(effects
 				(font
@@
 		)
 		(property "Footprint" "Resistor_THT:R_Axial_DIN0207_L6.3mm_D2.5mm_P7.62mm_Horizontal"
-			(at 90.17 70.358 90)
+			(at 78.232 72.39 90)
 			(effects
 				(font
@@
 		)
 		(property "Datasheet" "~"
-			(at 90.17 68.58 0)
+			(at 80.01 72.39 0)
 			(effects
 				(font
@@
 		)
 		(property "Description" "Resistor"
-			(at 90.17 68.58 0)
-			(effects
-				(font
+			(at 80.01 72.39 0)
+			(effects
+				(font
