File: hospital_traversing_robot/Electronics/station_circuit/station_circuit.kicad_sch (KiCad schematic)
At the start: 21 parts, among them J1 Barrel_Jack_MountingPin, SW1 switch, SW2 SW_Push, U1 Pico, U2 NRF24L01_Breakout, U3 LM338T

Commit message: further development in hospital rover project
Parts:
- removed SW1: switch, Connector_PinHeader_2.54mm:PinHeader_1x03_P2.54mm_Vertical, symbol Switch:SW_Nidec_CAS-120A1
Connections:
- net +3.3VP is gone; now on net +3.3V: U2.2 (VCC)
- net GND: now also U2.1 (GND)
- net +3.3VA: no longer names the net of U1.36 (3V3)
- net GNDA: no longer names the net of SW2.2, U1.28 (GND)
- net GNDA: no longer U2.1 (GND)
