File: product_display_stepper_speaker/Circuit/V2/V2.kicad_pcb (KiCad board)
At the start: 2 copper layers, 18 parts, among them J1 Barrel_Jack_MountingPin, SW1 SW_Push, U1 LM338T, U3 Pico

Commit message: finished product display stepper speaker circuit V2 PCB layout and generated gerber files and PDFs
Parts:
- added H1: MountingHole, MountingHole:MountingHole_3.2mm_M3, F.Cu at (84.9, 68.2)
- added H2: MountingHole, MountingHole:MountingHole_3.2mm_M3, F.Cu at (167.8, 114.7)
- J1: value Barrel_Jack_MountingPin -> Barrel_Jack
- R2: value 150 -> 470
- moved C1 44.4 mm to (137.8, 106.9), turned to 90 degrees
- moved R3 14.8 mm to (157.1, 80.0)
- moved R4 14.8 mm to (157.1, 83.2)
- moved MotionSensor1 14.4 mm to (168.9, 81.2)
- moved Speaker1 13.7 mm to (169.1, 93.1)
- moved Speaker2 13.7 mm to (169.1, 102.7)
- moved PAM8403_POT_breakout_board1 13.7 mm to (144.5, 90.7)
- moved R2 8.20 mm to (143.1, 78.1), turned to 90 degrees
- moved Stepper1 5.75 mm to (85.9, 86.0)
- moved A1 5.75 mm to (98.3, 82.3)
- moved Stepper2 5.00 mm to (86.2, 109.6)
- moved A2 5.00 mm to (98.3, 106.0)
- moved C2 4.86 mm to (86.1, 95.7)
- moved U3 3.75 mm to (118.5, 92.3)
- moved J1 3.22 mm to (156.8, 72.0)
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Connections:
- A2 pad 2: +5V -> unconnected-(A2-~{FLT}-Pad2)
- U3 pad 14: EN1 -> DIR1
- U3 pad 16: DIR1 -> EN1
- U3 pad 22: unconnected-(U3-GPIO17-Pad22) -> speaker_l
- U3 pad 24: unconnected-(U3-GPIO18-Pad24) -> speaker_r
- U3 pad 25: unconnected-(U3-GPIO19-Pad25) -> MotionSensor
- U3 pad 4: EN2 -> DIR2
- U3 pad 6: DIR2 -> EN2
Routing:
- net GND: track 4.18 -> 278.8 mm
- net +5V: track 0.00 -> 198.1 mm
- net +12V: track 0.00 -> 140.0 mm
- net MotionSensor: track 3.15 -> 49.0 mm
- net speaker_r: track 0.00 -> 18.0 mm
- net speaker_l: track 0.00 -> 18.0 mm
- net EN2: track 0.00 -> 13.7 mm
- net EN1: track 0.00 -> 11.5 mm
- net Net-(U1-ADJ): track 0.00 -> 8.57 mm
- net Net-(SW1-Pad2): track 3.99 -> 11.5 mm
- net Net-(U3-RUN): track 4.02 -> 11.5 mm
- net STEP1: track 0.00 -> 6.83 mm
- net DIR1: track 0.00 -> 6.83 mm
- net DIR2: track 0.00 -> 6.11 mm
- net STEP2: track 0.00 -> 6.11 mm
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Other:
- board outline added: 91.9 x 55.6 mm
