File: hospital_traversing_robot/Electronics/rover_circuit/Circuit.kicad_sch (KiCad schematic)
At the start: 30 parts, among them J1 Barrel_Jack, U1 L7805, U2 L298N, U3 LD33v, U4 NRF24L01_Breakout

Commit message: finished advanced movement component and some fine tuning
Other:
- note added: "TODOs: add power switch for battery add motor current sensing using ADC add beefier decoupling capacitors use better regulator for 3.3v (LM388) use mosfet and dtr pin for easy programming use jst for stc debug pins use better magnetometer"
Changed lines of the file:
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@@
 	(generator_version "9.0")
 	(paper "A4")
+	(text "TODOs:\nadd power switch for battery\nadd motor current sensing using ADC\nadd beefier decoupling capacitors\nuse better regulator for 3.3v (LM388)\nuse mosfet and dtr pin for easy programming\nuse jst for stc debug pins\nuse better magnetometer\n"
+		(exclude_from_sim no)
+		(at 235.966 58.928 0)
+		(effects
+			(font
+				(size 1.27 1.27)
+			)
+		)
+	)
 	(junction
 		(at 171.45 69.85)
