File: web_controlled_relay_board_v2.0/Electronics/Electronics.kicad_sch (KiCad schematic)
At the start: 69 parts, among them J1 Screw_Terminal_01x10, J2 Screw_Terminal_01x10, J3 Screw_Terminal_01x02, J4 Screw_Terminal_01x02, K1 G3MB-202P, K10 G3MB-202P, K11 G3MB-202P, K12 G3MB-202P, K13 G3MB-202P, K14 G3MB-202P, K15 G3MB-202P, K16 G3MB-202P, K17 G3MB-202P, K18 G3MB-202P, K19 G3MB-202P, K2 G3MB-202P, K20 G3MB-202P, K3 G3MB-202P, K4 G3MB-202P, K5 G3MB-202P, K6 G3MB-202P, K7 G3MB-202P, K8 G3MB-202P, K9 G3MB-202P, SW1 SW_MEC_5E, U1 PC817, U10 PC817, U11 PC817, U12 PC817, U13 PC817, U14 PC817, U15 PC817, U16 PC817, U17 PC817, U18 PC817, U19 PC817, U2 PC817, U20 PC817, U3 PC817, U4 PC817, U5 PC817, U6 PC817, U7 PC817, U8 PC817, U9 PC817

Commit message: PCB finished, pending final touches
Parts:
- J1, J2: footprint (none) -> TerminalBlock_CUI:TerminalBlock_CUI_TB007-508-10_1x10_P5.08mm_Horizontal
Connections:
- net AC: now also J4.1 (Pin_1), PS2.2 (AC/N); no longer J4.2 (Pin_2), PS2.1 (AC/L)
- net Control0: now also A1.25 (GPIO19); no longer A1.1 (GPIO0)
- net Control1: now also A1.24 (GPIO18); no longer A1.2 (GPIO1)
- net Control10: now also A1.12 (GPIO9); no longer A1.14 (GPIO10)
- net Control11: now also A1.11 (GPIO8); no longer A1.15 (GPIO11)
- net Control12: now also A1.10 (GPIO7); no longer A1.16 (GPIO12)
- net Control13: now also A1.9 (GPIO6); no longer A1.17 (GPIO13)
- net Control14: now also A1.7 (GPIO5); no longer A1.19 (GPIO14)
- net Control15: now also A1.6 (GPIO4); no longer A1.20 (GPIO15)
- net Control16: now also A1.5 (GPIO3); no longer A1.21 (GPIO16)
- net Control17: now also A1.4 (GPIO2); no longer A1.22 (GPIO17)
- net Control18: now also A1.2 (GPIO1); no longer A1.24 (GPIO18)
- net Control19: now also A1.1 (GPIO0); no longer A1.25 (GPIO19)
- net Control2: now also A1.22 (GPIO17); no longer A1.4 (GPIO2)
- net Control3: now also A1.21 (GPIO16); no longer A1.5 (GPIO3)
- net Control4: now also A1.20 (GPIO15); no longer A1.6 (GPIO4)
- net Control5: now also A1.19 (GPIO14); no longer A1.7 (GPIO5)
- net Control6: now also A1.17 (GPIO13); no longer A1.9 (GPIO6)
- net Control7: now also A1.16 (GPIO12); no longer A1.10 (GPIO7)
- net Control8: now also A1.15 (GPIO11); no longer A1.11 (GPIO8)
- net Control9: now also A1.14 (GPIO10); no longer A1.12 (GPIO9)
- net NEUT: now also J4.2 (Pin_2), PS2.1 (AC/L); no longer J4.1 (Pin_1), PS2.2 (AC/N)
- net at U2.1: now also R1.2; no longer R2.2
- net at PowerPin1.2 (Pin_2): now also A1.39 (VSYS)
- net at U1.1: now also R2.2; no longer R1.2
Other:
- moved on the sheet: J4, PowerPin1, R1, R2

Commit message: finished final touches of PCB schematic and layout
Parts:
- added C1: C_Polarized, Capacitor_THT:CP_Radial_D6.3mm_P2.50mm, symbol Device:C_Polarized
- added C2: C_Polarized, Capacitor_THT:CP_Radial_D8.0mm_P3.50mm, symbol Device:C_Polarized
Connections:
- net +3.3V: now also C1.1
- net +5V: now also C2.1
- net GND: now also C2.2
- net GNDA: now also C1.2
Other:
- moved on the sheet: A1, J4, PS1, PS2, PowerPin1, SW1
